File: BBBBoat-cape.brd (EAGLE design)
At the start: 54.6 x 71.8 mm, 34 parts

Commit message: change PWM pin
the pwm B pins currently don't work in the PyBBIO library
so PWM2B was switched to PWM1A
Connections:
- new net PWM_SWITCH: U$1.60
Changed lines of the file:
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@@
 <wire x1="44.704" y1="61.087" x2="44.704" y2="58.674" width="0.6096" layer="1"/>
+</signal>
+<signal name="PWM_SWITCH">
+<contactref element="U$1" pad="60"/>
 </signal>
 </signals>
